File: Design/Controller/NixieController.kicad_pcb (KiCad board)
At the start: 2 copper layers, 180 x 41 mm, 104 parts, among them J1 Conn_01x12_Female, J2 Conn_01x12_Female, J3 Conn_01x12_Female, J4 Conn_01x12_Female, J5 Conn_01x12_Female, J6 Conn_01x12_Female, J7 Jack-DC, J8 Conn_01x02_Male, J9 Conn_01x06_Male, Q1 IRF644, Q10 BSS127, Q11 BSS127, Q12 BSS127, Q13 BSS127, Q14 BSS127, Q15 BSS127, Q16 BSS127, Q17 BSS127, Q18 BSS127, Q19 BSS127, Q2 BSS127, Q20 BSS127, Q21 BSS127, Q22 BSS127, Q23 BSS127, Q24 BSS127, Q25 BSS127, Q26 BSS127, Q27 BSS127, Q28 BSS127, Q29 BSS127, Q3 BSS127, Q30 BSS127, Q31 BSS127, Q32 BSS127, Q33 BSS127, Q34 BSS127, Q35 BSS127, Q36 BSS127, Q37 BSS127, Q38 BSS127, Q39 BSS127, Q4 BSS127, Q40 BSS127, Q41 BSS127, Q42 BSS127, Q43 BSS127, Q44 BSS127, Q45 BSS127, Q46 BSS127, Q47 BSS127, Q48 BSS127, Q49 BSS127, Q5 BSS127, Q50 BSS127, Q51 BSS127, Q52 BSS127, Q53 BSS127, Q54 BSS127, Q55 BSS127, Q56 BSS127, Q57 BSS127, Q58 BSS127, Q59 BSS127, Q6 BSS127, Q60 BSS127, Q61 BSS127, Q7 BSS127, Q8 BSS127, Q9 BSS127, U1 ATtiny85-20SU, U10 74HC595, U11 74HC595, U12 74HC595, U2 DS1307Z+, U3 LM2576, U4 MAX1771, U5 74HC595, U6 74HC595, U7 74HC595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

Commit message: Add license notice to all human readable files
Other:
- board text added: "Nixie Controller PCB Copyright (C) 2020 Daniel He See <https://www.gnu.org/licenses/>."
- board text added: "Nixie Controller PCB Copyright (C) 2020 Daniel He This program is free software: you can redistribute it and/or modify it under the terms of the GNU General Public License as published by the Free Software Foundation, either version 3 of the License, or (at your option) any later version. This program is distributed in the hope that it will be useful, but WITHOUT ANY WARRANTY; without even the im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"
