File: Design/Sockets/IN-18/IN-18.kicad_pcb (KiCad board)
At the start: 2 copper layers, 245 x 50 mm, 19 parts, among them J1 Conn_01x12_Male, J2 Conn_01x12_Male, J3 Conn_01x12_Male, J4 Conn_01x12_Male, J5 Conn_01x12_Male, J6 Conn_01x12_Male, U1 IN-18, U2 IN-18, U3 IN-18, U4 IN-18, U5 IN-18, U6 IN-18

Commit message: Add front copper plane to IN-18 socket board, increase clearance, add high voltage warning symbol
Parts:
- added REF**: Symbol_HighVoltage_Type2_CopperTop_VerySmall, Symbol:Symbol_HighVoltage_Type2_CopperTop_VerySmall, F.Cu at (10.0, 76.0)
Routing:
- added copper zone on F.Cu, net GND
Other:
- board text added: "HIGH VOLTAGE"

Commit message: Add license notice to all human readable files
Other:
- board text added: "IN-18 Nixie Socket PCB Copyright (C) 2020 Daniel He See <https://www.gnu.org/licenses/>."
- board text added: "IN-18 Nixie Socket PCB Copyright (C) 2020 Daniel He This program is free software: you can redistribute it and/or modify it under the terms of the GNU General Public License as published by the Free Software Foundation, either version 3 of the License, or (at your option) any later version. This program is distributed in the hope that it will be useful, but WITHOUT ANY WARRANTY; without even the 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"
